File: Hardware/TT7D v1.0.brd (EAGLE design)
At the start: 25 x 55 mm, 49 parts, among them U1 ATMEGA328P-AU, U2 UBLOX_MAX-7C, U3 SI406X, U4 IT3205CE_TCXO_6P, U5 MCP1640

Commit message: Add files via upload
Other:
- board text added: "JLCJLCJLCJLC"
Changed lines of the file:
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@@
 <wire x1="11.65" y1="32" x2="11.65" y2="30" width="0.1524" layer="22"/>
 <rectangle x1="18.25" y1="39" x2="20.25" y2="42" layer="30"/>
+<text x="17.25" y="33" size="0.81" layer="21" font="vector" ratio="20" rot="R90">JLCJLCJLCJLC</text>
 </plain>
 <attributes>
