File: Hardware/TT7D v1.0.sch (EAGLE design)
At the start: 49 parts, among them U1 ATMEGA328P-AU, U2 UBLOX_MAX-7C, U3 SI406X, U4 IT3205CE_TCXO_6P, U5 MCP1640

Commit message: Add files via upload
Other:
- note added: "RC filter: L2=10kΩ, C8=2.4pF, C9=NC"
- note added: "Voltage Divider: R6=4.7kΩ, R5=10kΩ"
Changed lines of the file:
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@@
 <text x="345.44" y="58.42" size="1.778" layer="94">3.3V operating voltage, power source: AAA primary cell.</text>
 <text x="345.44" y="55.88" size="1.778" layer="94">Optionally solar powered - two cells instead of battery.</text>
+<text x="116.84" y="22.86" size="1.778" layer="94">RC filter: L2=10kΩ, C8=2.4pF,  C9=NC</text>
+<text x="116.84" y="20.32" size="1.778" layer="94">Voltage Divider: R6=4.7kΩ, R5=10kΩ</text>
 </plain>
 <instances>

Commit message: Add files via upload
Other:
- note added: "RC filter: L2=R=4.7kΩ, C8=2.4pF, C9=NC"
- note added: "Voltage Divider: R6=NC, R5=0Ω"
- note removed: "RC filter: L2=10kΩ, C8=2.4pF, C9=NC"
- note removed: "Voltage Divider: R6=4.7kΩ, R5=10kΩ"
Changed lines of the file:
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@@
 <text x="345.44" y="58.42" size="1.778" layer="94">3.3V operating voltage, power source: AAA primary cell.</text>
 <text x="345.44" y="55.88" size="1.778" layer="94">Optionally solar powered - two cells instead of battery.</text>
-<text x="116.84" y="22.86" size="1.778" layer="94">RC filter: L2=10kΩ, C8=2.4pF,  C9=NC</text>
-<text x="116.84" y="20.32" size="1.778" layer="94">Voltage Divider: R6=4.7kΩ, R5=10kΩ</text>
+<text x="116.84" y="22.86" size="1.778" layer="94">RC filter: L2=R=4.7kΩ, C8=2.4pF,  C9=NC</text>
+<text x="116.84" y="20.32" size="1.778" layer="94">Voltage Divider: R6=NC, R5=0Ω</text>
 </plain>
 <instances>

Commit message: Add files via upload
Other:
- note added: "23.11.2019 22:00"
- note added: "A low-cost APRS/RTTY balloon"
- note added: "ATMEGA328P - Microcontroller"
- note added: "MAX-M8Q - GNSS"
- note added: "MCP1640 - Boost Converter"
- note added: "Si4x6x - Transmitter"
- note added: "TT7D Tracker v1.0"
- note added: "Tomas (TT7)"
- note added: "https://tt7hab.blogspot.com/"
- note added: "primary battery or a pair of"
- note added: "solar cells."
- note added: "tracker. Powered by a AAA"
- note removed: "3.3V operating voltage, power source: AAA primary cell."
- note removed: "APRS / RTTY high altitude balloon tracker."
- note removed: "ATmega328P"
- note removed: "Optionally solar powered - two cells instead of battery."
- note removed: "Si4060 / Si4063 / Si4460 / Si4463"
- note removed: "TT7D Tracker"
- note removed: "u-blox MAX-M8Q"
- moved on the sheet: C0, C1, C10, C11, C12, C13, C14, C15, C2, C3, C4, C5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
